File: elecsoc_card.kicad_sch (KiCad schematic)
At the start: 35 parts, among them J1 Conn_01x02_Pin, J2 Conn_01x02_Pin, U1 NA555D

Commit message: Added soldering instructions
Other:
- note added: "If all components placed, result is the original period T = 0.693*(R1/2+2*R2/2)*C1*2 = 0.693*(R1+2*R2)*C1"
- note added: "If optional caps added: T = 0.693*(R1+2*R2)*C1 = 0.693 * 3 * 78.7k * 10u = 1.636s T = 0.693*(R1+2*R2)*(C1+C3) = 0.693 * 3 * 78.7k * 20u = 3.272s"
- note added: "If optional resistors added: T = 0.693*(R1+2*R2)*C1 = 0.693 * 3 * 78.7k * 10u = 1.636s T = 0.693*(R1/2+2*R2/2)*C1 = 0.693 * 3 * 78.7k/2 * 10u = 0.818s"
- note added: "T = 0.693*(R1+2*R2)*C1 = 0.693 * 3 * 78.7k * 10u = 1.636s"
- note removed: "If all components placed, result is the original period T = 0.693*(R1/2+2*R2/2)*(C1+C2) = 0.693 * 3 * 40k * 20u = 1.663s"
- note removed: "If optional caps added: T = 0.693*(R1+2*R2)*C1 = 0.693 * 3 * 50k * 10u = 1.663s T = 0.693*(R1+2*R2)*(C1+C3) = 0.693 * 3 * 50k * 20u = 3.326s"
- note removed: "If optional resistors added: T = 0.693*(R1+2*R2)*C1 = 0.693 * 3 * 50k * 10u = 1.663s T = 0.693*(R1/2+2*R2/2)*C1 = 0.693 * 3 * 40k * 10u = 0.832s"
- note removed: "T = 0.693*(R1+2*R2)*C1 = 0.693 * 3 * 10k * 47u = 0.97s"
- note removed: "T = 0.693*(R1+2*R2)*C1 = 0.693 * 3 * 4.99k * 47u = 0.487s"
- note removed: "T = 0.693*(R1+2*R2)*C1 = 0.693 * 3 * 50k * 10u = 1.04s"
- company: ElecSoc -> JayceDesign
- title: ElecSoc USB business card -> ElecSoc Soldering Practice Card
Changed lines of the file:
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@@
 	(paper "A4")
 	(title_block
-		(title "ElecSoc USB business card")
-		(company "ElecSoc")
+		(title "ElecSoc Soldering Practice Card")
+		(date "2024-08-14")
+		(company "JayceDesign")
 	)
 	(junction
@@
 	(text "RED Leds\nVf = 3V\nIf = 5mA\nRled = (Vs - Vf)/If = (5 - 3)/0.005 = 400\n\nWhite Leds\nVf = 2.9\nIf = 5m\nRled = (Vs - Vf)/If = (5 - 2.9)/0.005 = 420"
 		(exclude_from_sim no)
-		(at 231.648 103.124 0)
-		(effects
-			(font
-				(size 1.27 1.27)
-			)
-			(justify left bottom)
-		)
-	)
-	(text "T = 0.693*(R1+2*R2)*C1\n  = 0.693 * 3 * 50k * 10u \n  = 1.04s"
-		(exclude_from_sim no)
-		(at 232.41 82.55 0)
-		(effects
-			(font
-				(size 1.27 1.27)
-			)
-			(justify left bottom)
-		)
-	)
-	(text "If optional resistors added:\nT = 0.693*(R1+2*R2)*C1\n  = 0.693 * 3 * 50k * 10u \n  = 1.663s\nT = 0.693*(R1/2+2*R2/2)*C1\n  = 0.693 * 3 * 40k * 10u \n  = 0.832s"
-		(exclude_from_sim no)
-		(at 231.902 135.89 0)
+		(at 22.86 70.612 0)
+		(effects
+			(font
+				(size 1.27 1.27)
+			)
+			(justify left bottom)
+		)
+	)
+	(text "If optional resistors added:\nT = 0.693*(R1+2*R2)*C1\n  = 0.693 * 3 * 78.7k * 10u \n  = 1.636s\nT = 0.693*(R1/2+2*R2/2)*C1\n  = 0.693 * 3 * 78.7k/2 * 10u \n  = 0.818s"
+		(exclude_from_sim no)
+		(at 228.346 115.824 0)
 		(effects
 			(font
@@
 		)
 	)
-	(text "If optional caps added:\nT = 0.693*(R1+2*R2)*C1\n  = 0.693 * 3 * 50k * 10u \n  = 1.663s\nT = 0.693*(R1+2*R2)*(C1+C3)\n  = 0.693 * 3 * 50k * 20u \n  = 3.326s"
-		(exclude_from_sim no)
-		(at 231.394 119.888 0)
+	(text "If optional caps added:\nT = 0.693*(R1+2*R2)*C1\n  = 0.693 * 3 * 78.7k * 10u \n  = 1.636s\nT = 0.693*(R1+2*R2)*(C1+C3)\n  = 0.693 * 3 * 78.7k * 20u \n  = 3.272s"
+		(exclude_from_sim no)
+		(at 228.6 99.822 0)
 		(effects
 			(font
@@
 		)
 	)
-	(text "T = 0.693*(R1+2*R2)*C1\n  = 0.693 * 3 * 10k * 47u \n  = 0.97s"
-		(exclude_from_sim no)
-		(at 232.41 73.66 0)
-		(effects
-			(font
-				(size 1.27 1.27)
-			)
-			(justify left bottom)
-		)
-	)
 	(text "Pin Headers"
 		(exclude_from_sim no)
@@
 	(text "Resistors and capacitance values for oscillator"
 		(exclude_from_sim no)
-		(at 232.41 58.42 0)
-		(effects
-			(font
-				(size 1.27 1.27)
-			)
-			(justify left bottom)
-		)
-	)
-	(text "If all components placed, result is the original period\nT = 0.693*(R1/2+2*R2/2)*(C1+C2)\n  = 0.693 * 3 * 40k * 20u \n  = 1.663s"
-		(exclude_from_sim no)
-		(at 231.14 144.78 0)
+		(at 229.362 77.216 0)
+		(effects
+			(font
+				(size 1.27 1.27)
+			)
+			(justify left bottom)
+		)
+	)
+	(text "If all components placed, result is the original period\nT = 0.693*(R1/2+2*R2/2)*C1*2\n  = 0.693*(R1+2*R2)*C1"
+		(exclude_from_sim no)
+		(at 228.092 124.206 0)
 		(effects
 			(font
@@
 		)
 	)
-	(text "T = 0.693*(R1+2*R2)*C1\n  = 0.693 * 3 * 4.99k * 47u \n  = 0.487s"
-		(exclude_from_sim no)
-		(at 232.41 64.77 0)
-		(effects
-			(font
+	(text "T = 0.693*(R1+2*R2)*C1\n  = 0.693 * 3 * 78.7k * 10u \n  = 1.636s"
+		(exclude_from_sim no)
+		(at 229.362 83.566 0)
+		(effects
+			(font
